File: HW/Controller.sch (KiCad schematic (older format))
At the start: 24 parts, among them J1 Spare, J2 +12V_con, J3 LimitUpper, J4 ControlSwitch, J5 LimitLower, J6 Motor_controller_connections, U1 L7805, U2 ATMEGA328P-AU-Arduino, Y1 8MHZ

Commit message: PCB
Parts:
- 1U1, C1, C5, C6, C7, C8, C9: symbol C -> device:C
- C2: symbol CP_Small -> device:CP_Small
- C3: symbol CP -> device:CP
- C4: symbol C_Small -> device:C_Small
- D1: symbol WS2812B -> WS2812B:WS2812B
- F1: symbol Polyfuse -> device:Polyfuse
- FTDI1: symbol CONN_01X06 -> Controller-rescue:CONN_01X06
- J1: symbol Conn_01x04 -> conn:Conn_01x04
- J2: symbol Screw_Terminal_01x02 -> conn:Screw_Terminal_01x02
- J3, J4, J5: symbol Screw_Terminal_01x03 -> conn:Screw_Terminal_01x03
- J6: symbol Screw_Terminal_01x09 -> conn:Screw_Terminal_01x09
- JP1: symbol Jumper -> device:Jumper
- R1: symbol R -> device:R
- U1: symbol L7805 -> regul:L7805
- U2: symbol ATMEGA328P-AU-Arduino -> Peters:ATMEGA328P-AU-Arduino
- Y1: symbol Crystal -> device:Crystal
